File: bl_motor_dora3/bl_dora2.brd (EAGLE design)
At the start: 85 x 50.8 mm, 78 parts

Commit message: Add files via upload
Parts:
- added C13, C14, C15, C16, C17, C18: 5n, rcl:C2012
- added U$19: XH_2P, user:XH_2P
- added U$20, U$21, U$22, U$26, U$27, U$28: ES3BB13F, user:ES3BB13F
- C5, C6, C7: value 0.1u -> 0.22u
- R15: value 100k -> 33k
- R18, R19, R20, R21, R22, R23: value 47 -> 10
- R26, R30, R31, R32, R6, R7: device rcl:R2512 -> rcl:R1206
- R29: value 10jk -> 10k
- R3, R4: value 4.7k -> 10k
- moved R32 148.8 mm to (54.9, 34.3), flipped to the bottom, turned to 180 degrees
- moved R31 132.2 mm to (55.0, 20.2), flipped to the bottom, turned to 180 degrees
- moved F_C5 125.0 mm to (68.7, 32.9), flipped to the bottom
- moved R6 121.8 mm to (54.9, 32.1), flipped to the bottom, turned to 180 degrees
- moved R30 117.8 mm to (54.9, 7.49), flipped to the bottom, turned to 180 degrees
- moved R7 116.3 mm to (55.0, 18.0), flipped to the bottom, turned to 180 degrees
- moved F_C6 115.7 mm to (48.3, 32.6), flipped to the bottom
- moved F_C4 112.4 mm to (68.6, 18.9), flipped to the bottom
- moved R26 111.7 mm to (54.9, 5.21), flipped to the bottom, turned to 180 degrees
- moved F_C3 103.6 mm to (68.5, 5.21), flipped to the bottom
- moved U$17 88.2 mm to (62.5, 9.14), turned to 270 degrees
- moved F_C2 86.2 mm to (48.3, 18.7), flipped to the bottom
- moved U$16 85.5 mm to (62.4, 23.1), turned to 270 degrees
- moved F_C1 79.7 mm to (48.1, 5.46), flipped to the bottom
- moved U$13 76.5 mm to (62.5, 37.1), turned to 270 degrees
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Connections:
- removed net N$39: F_C1.P$1, R32.1, U$18.K
- removed net N$4: C5.2, F_C3.P$2, N$20N$21.1, R32.2, U$1.PIN25, U$11.PIN3_S, U$12.PIN2_D, U$18.A1, U$18.A2, U$25.P$3
- removed net N$8: F_C1.P$2, F_C2.P$2, F_C6.P$2, R11.2, R12.2, R13.2, R14.2, R27.1, R28.1, R29.1, U$1.PIN21, U$1.PIN38, U$10.PIN3_S, U$12.PIN3_S, U$8.PIN3_S
- removed net N$9: F_C6.P$1, R6.1, U$14.K
- new net N$41: F_C3.P$2, R30.2, U$22.A
- new net N$44: C17.2, C5.2, N$20N$21.1, U$1.PIN25, U$11.PIN3_S, U$12.PIN2_D, U$17.A1, U$17.A2, U$18.K, U$22.C, U$25.P$3, U$28.A
- new net N$45: F_C1.P$1, R26.1, U$28.C
- new net N$47: F_C2.P$1, R7.1, U$27.C
- net GND: now also U$1.PIN21, U$19.P$1; no longer U$1.PIN22
- net N$19: now also C13.2, U$13.A1, U$13.A2, U$14.K, U$20.C, U$26.A; no longer F_C5.P$2, R6.2, U$14.A1, U$14.A2
- net N$25: now also C13.1
- net N$26: now also C18.1
- net N$27: now also C17.1
- net N$28: now also C16.1
- net N$29: now also C15.1
- net N$30: now also C14.1
- net N$38: now also F_C4.P$2, R31.2, U$21.A; no longer F_C2.P$1, R26.1, U$15.K
- net N$40: now also C14.2, C15.2, C16.2, F_C1.P$2, F_C2.P$2, F_C6.P$2, R11.2, R12.2, R13.2, R14.2, R27.1, R28.1, R29.1, R30.1, R32.1, U$1.PIN22, U$1.PIN38, U$10.PIN3_S, U$12.PIN3_S, U$14.A1, U$14.A2, U$15.A1, U$15.A2, U$18.A1, U$18.A2, U$8.PIN3_S; no longer F_C3.P$1, U$17.K
- net N$42: now also F_C6.P$1, R6.1, U$26.C; no longer F_C4.P$1, R30.1, U$16.K
- net N$5: now also F_C5.P$2, R32.2, U$20.A; no longer F_C5.P$1, R7.1, U$13.K
- net N$50: now also C18.2, U$15.K, U$16.A1, U$16.A2, U$21.C, U$27.A; no longer F_C4.P$2, R26.2, U$15.A1, U$15.A2
- net VCC: now also F_C3.P$1, F_C4.P$1, F_C5.P$1, R26.2, R6.2, U$13.K, U$16.K, U$17.K, U$19.P$2; no longer R30.2, R31.2, U$13.A1, U$13.A2, U$16.A1, U$16.A2, U$17.A1, U$17.A2
Routing:
- net N$40: track 0.00 -> 140.0 mm, vias 0 -> 67
- net N$8: track 107.8 -> 0.00 mm, vias 37 -> 0
- net N$44: track 0.00 -> 101.1 mm, vias 0 -> 76
- net N$4: track 79.1 -> 0.00 mm, vias 61 -> 0
- net GND: track 73.1 -> 137.1 mm, vias 15 -> 53
- net N$19: track 74.0 -> 88.9 mm, vias 53 -> 60
- net N$50: track 75.5 -> 85.0 mm, vias 3 -> 57
- net N$38: track 0.00 -> 8.99 mm, vias 0 -> 1
- net N$5: track 0.00 -> 8.94 mm, vias 0 -> 1
- net N$41: track 0.00 -> 8.27 mm, vias 0 -> 1
- net N$45: track 0.00 -> 6.84 mm
- net N$35: track 45.1 -> 51.8 mm, vias 3 -> 1
- net N$47: track 0.00 -> 6.68 mm
- net N$36: track 36.4 -> 43.0 mm
- net N$42: track 0.00 -> 6.53 mm
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- added copper zone on layer 1, net N$40
- added copper zone on layer 16, net N$40
- added copper zone on layer 1, net N$44
- added copper zone on layer 16, net N$44
- added copper zone on layer 1, net N$50
- added copper zone on layer 16, net N$50
- removed copper zone on layer 1, net N$20
- removed copper zone on layer 16, net N$20
- removed copper zone on layer 1, net N$4
- removed copper zone on layer 16, net N$4
- removed copper zone on layer 1, net N$8
- removed copper zone on layer 16, net N$8
Other:
- board text added: "BL_MotaDora-Mod.1"
- board text added: "KRP"
- board text removed: "BL_MotaDora-Mod.2"
- board text removed: "vcc"
