File: bl_motor_dora3/bl_dora2.sch (EAGLE design)
At the start: 78 parts

Commit message: Add files via upload
Parts:
- added C13, C14, C15, C16, C17, C18: 5n, rcl:C-EUC2012
- added U$19: XH_2P, user:XH_2P
- added U$20, U$21, U$22, U$26, U$27, U$28: ES3BB13F, user:ES3BB13F
- C5, C6, C7: value 0.1u -> 0.22u
- R15: value 100k -> 33k
- R18, R19, R20, R21, R22, R23: value 47 -> 10
- R26, R30, R31, R32, R6, R7: device rcl:R-EU_R2512 -> rcl:R-EU_R1206
- R29: value 10jk -> 10k
- R3, R4: value 4.7k -> 10k
Connections:
- removed net N$39: F_C1.1, R32.1, U$18.K
- removed net N$4: C5.2, F_C3.2, N$20N$21.1, R32.2, U$1.PIN25_SC, U$11.PIN3_S, U$12.PIN2_D, U$18.A1, U$18.A2, U$25.PIN3
- removed net N$8: F_C1.2, F_C2.2, F_C6.2, R11.2, R12.2, R13.2, R14.2, R27.1, R28.1, R29.1, U$1.PIN21_CSN, U$1.PIN38_LSS, U$10.PIN3_S, U$12.PIN3_S, U$8.PIN3_S
- removed net N$9: F_C6.1, R6.1, U$14.K
- new net N$41: F_C3.2, R30.2, U$22.A
- new net N$44: C17.2, C5.2, N$20N$21.1, U$1.PIN25_SC, U$11.PIN3_S, U$12.PIN2_D, U$17.A1, U$17.A2, U$18.K, U$22.C, U$25.PIN3, U$28.A
- new net N$45: F_C1.1, R26.1, U$28.C
- new net N$47: F_C2.1, R7.1, U$27.C
- net GND: now also U$1.PIN21_CSN, U$19.P$1; no longer U$1.PIN22_CSP
- net N$19: now also C13.2, U$13.A1, U$13.A2, U$14.K, U$20.C, U$26.A; no longer F_C5.2, R6.2, U$14.A1, U$14.A2
- net N$25: now also C13.1
- net N$26: now also C18.1
- net N$27: now also C17.1
- net N$28: now also C16.1
- net N$29: now also C15.1
- net N$30: now also C14.1
- net N$38: now also F_C4.2, R31.2, U$21.A; no longer F_C2.1, R26.1, U$15.K
- net N$40: now also C14.2, C15.2, C16.2, F_C1.2, F_C2.2, F_C6.2, R11.2, R12.2, R13.2, R14.2, R27.1, R28.1, R29.1, R30.1, R32.1, U$1.PIN22_CSP, U$1.PIN38_LSS, U$10.PIN3_S, U$12.PIN3_S, U$14.A1, U$14.A2, U$15.A1, U$15.A2, U$18.A1, U$18.A2, U$8.PIN3_S; no longer F_C3.1, U$17.K
- net N$42: now also F_C6.1, R6.1, U$26.C; no longer F_C4.1, R30.1, U$16.K
- net N$5: now also F_C5.2, R32.2, U$20.A; no longer F_C5.1, R7.1, U$13.K
- net N$50: now also C18.2, U$15.K, U$16.A1, U$16.A2, U$21.C, U$27.A; no longer F_C4.2, R26.2, U$15.A1, U$15.A2
- net VCC: now also F_C3.1, F_C4.1, F_C5.1, R26.2, R6.2, U$13.K, U$16.K, U$17.K, U$19.P$2; no longer R30.2, R31.2, U$13.A1, U$13.A2, U$16.A1, U$16.A2, U$17.A1, U$17.A2
Other:
- note added: "47Ωの抵抗器は1206の0.66W。rs品番721-9715"
- note added: "F_C*のコンデンサは0.1uFのフィルムコンデンサ"
- note added: "csnとcspはできるだけ同じ長さで同じルート・無理にくねくねさせるなら同じながさでなくていい"
- note added: "deadタイムは約600nsec"
- note added: "fetにSQD50034ELを使う。同じto252"
- note added: "fetのドレインソース間がオン時に1Vを超えたら短絡とみなされる"
- note added: "電流制限は30Aに設定されている。refの抵抗比を変えることで変更可"
- note removed: "csnとcspはできるだけ同じ長さで同じルート"
- note removed: "deadタイムは約1420nsec"
- moved on the sheet: F_C2, F_C3, F_C4, F_C5, F_C6, R10, R11, R12, R13, R14, R26, R30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
