File: bl_motor_dora3/bl_dora2.sch (EAGLE design)
At the start: 91 parts

Commit message: エンハンスドver
Parts:
- R10: value 47k -> 20k
- R5: value 22k -> 39k
- R8: value 39k -> 22k
- R9: value 10k -> 3.3k
- U$23: value ZH_6P -> ZH_6P_L; device user:ZH_6P -> user:ZH_6P_L
Changed lines of the file:
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@@
 <part name="AGND4" library="supply1" library_urn="urn:adsk.eagle:library:371" deviceset="AGND" device=""/>
 <part name="AGND6" library="supply1" library_urn="urn:adsk.eagle:library:371" deviceset="AGND" device=""/>
-<part name="R8" library="rcl" library_urn="urn:adsk.eagle:library:334" deviceset="R-EU_" device="M2012" package3d_urn="urn:adsk.eagle:package:23561/2" value="39k"/>
-<part name="R9" library="rcl" library_urn="urn:adsk.eagle:library:334" deviceset="R-EU_" device="M2012" package3d_urn="urn:adsk.eagle:package:23561/2" value="10k"/>
-<part name="R10" library="rcl" library_urn="urn:adsk.eagle:library:334" deviceset="R-EU_" device="M2012" package3d_urn="urn:adsk.eagle:package:23561/2" value="47k"/>
+<part name="R8" library="rcl" library_urn="urn:adsk.eagle:library:334" deviceset="R-EU_" device="M2012" package3d_urn="urn:adsk.eagle:package:23561/2" value="22k"/>
+<part name="R9" library="rcl" library_urn="urn:adsk.eagle:library:334" deviceset="R-EU_" device="M2012" package3d_urn="urn:adsk.eagle:package:23561/2" value="3.3k"/>
+<part name="R10" library="rcl" library_urn="urn:adsk.eagle:library:334" deviceset="R-EU_" device="M2012" package3d_urn="urn:adsk.eagle:package:23561/2" value="20k"/>
 <part name="AGND7" library="supply1" library_urn="urn:adsk.eagle:library:371" deviceset="AGND" device=""/>
 <part name="R11" library="rcl" library_urn="urn:adsk.eagle:library:334" deviceset="R-EU_" device="R2512" package3d_urn="urn:adsk.eagle:package:23545/2" value="20m"/>
@@
 <part name="U$2" library="user" deviceset="2SC5964" device=""/>
 <part name="U$5" library="user" deviceset="1005X4RESISTOR" device="" value="10K"/>
-<part name="U$23" library="user" deviceset="ZH_6P" device=""/>
 <part name="AGND16" library="supply1" library_urn="urn:adsk.eagle:library:371" deviceset="AGND" device=""/>
 <part name="AGND17" library="supply1" library_urn="urn:adsk.eagle:library:371" deviceset="AGND" device=""/>
@@
 <part name="JP4" library="pinhead" library_urn="urn:adsk.eagle:library:325" deviceset="PINHD-1X8" device="" package3d_urn="urn:adsk.eagle:package:22409/2"/>
 <part name="C12" library="rcl" library_urn="urn:adsk.eagle:library:334" deviceset="CPOL-EU" device="153CLV-1012" package3d_urn="urn:adsk.eagle:package:23404/2" value="820u"/>
-<part name="R5" library="rcl" library_urn="urn:adsk.eagle:library:334" deviceset="R-EU_" device="M2012" package3d_urn="urn:adsk.eagle:package:23561/2" value="22k"/>
+<part name="R5" library="rcl" library_urn="urn:adsk.eagle:library:334" deviceset="R-EU_" device="M2012" package3d_urn="urn:adsk.eagle:package:23561/2" value="39k"/>
 <part name="U$4" library="user" deviceset="RGB_LED" device=""/>
 <part name="AGND5" library="supply1" library_urn="urn:adsk.eagle:library:371" deviceset="AGND" device=""/>
@@
 <part name="R31" library="rcl" library_urn="urn:adsk.eagle:library:334" deviceset="R-EU_" device="R1206" package3d_urn="urn:adsk.eagle:package:23540/2" value="22"/>
 <part name="R32" library="rcl" library_urn="urn:adsk.eagle:library:334" deviceset="R-EU_" device="R1206" package3d_urn="urn:adsk.eagle:package:23540/2" value="22"/>
+<part name="U$23" library="user" deviceset="ZH_6P_L" device=""/>
 </parts>
 <sheets>
@@
 <attribute name="VALUE" x="-73.66" y="76.2" size="2.54" layer="96" rot="R180"/>
 </instance>
-<instance part="U$23" gate="G$1" x="-144.78" y="40.64" smashed="yes" rot="R270"/>
 <instance part="AGND16" gate="VR1" x="-129.54" y="22.86" smashed="yes">
 <attribute name="VALUE" x="-132.08" y="17.78" size="1.778" layer="96" rot="R90"/>
@@
 <attribute name="VALUE" x="341.122" y="113.03" size="1.778" layer="96" rot="R90"/>
 </instance>
+<instance part="U$23" gate="G$1" x="-144.78" y="40.64" smashed="yes" rot="R270"/>
 </instances>
 <busses>
@@
 </segment>
 <segment>
-<pinref part="U$23" gate="G$1" pin="PIN1"/>
 <wire x1="-139.7" y1="53.34" x2="-129.54" y2="53.34" width="0.1524" layer="91"/>
 <label x="-129.54" y="53.34" size="1.778" layer="95"/>
+<pinref part="U$23" gate="G$1" pin="PIN1"/>
 </segment>
 <segment>
@@
 </segment>
 <segment>
-<pinref part="U$23" gate="G$1" pin="PIN6"/>
 <wire x1="-139.7" y1="27.94" x2="-129.54" y2="27.94" width="0.1524" layer="91"/>
 <wire x1="-129.54" y1="27.94" x2="-129.54" y2="25.4" width="0.1524" layer="91"/>
 <pinref part="AGND16" gate="VR1" pin="AGND"/>
+<pinref part="U$23" gate="G$1" pin="PIN6"/>
 </segment>
 <segment>
@@
 </segment>
 <segment>
-<pinref part="U$23" gate="G$1" pin="PIN3"/>
 <wire x1="-139.7" y1="43.18" x2="-129.54" y2="43.18" width="0.1524" layer="91"/>
 <label x="-129.54" y="43.18" size="1.778" layer="95"/>
+<pinref part="U$23" gate="G$1" pin="PIN3"/>
 </segment>
 </net>
@@
 </segment>
 <segment>
-<pinref part="U$23" gate="G$1" pin="PIN4"/>
 <wire x1="-139.7" y1="38.1" x2="-129.54" y2="38.1" width="0.1524" layer="91"/>
 <label x="-129.54" y="38.1" size="1.778" layer="95"/>
+<pinref part="U$23" gate="G$1" pin="PIN4"/>
 </segment>
 </net>
@@
 </segment>
 <segment>
-<pinref part="U$23" gate="G$1" pin="PIN5"/>
 <wire x1="-139.7" y1="33.02" x2="-129.54" y2="33.02" width="0.1524" layer="91"/>
 <label x="-129.54" y="33.02" size="1.778" layer="95"/>
-</segment>
-</net>
+<pinref part="U$23" gate="G$1" pin="PIN5"/>
+</segment>
+</net>

Commit message: シャント抵抗ラインにローパスフィルタの追加
電流制限、電流測定がつかいもんにならんかったからノイズを消すためにローパスフィルタをシャント抵抗の電位差を測るラインに追加
Parts:
- added C19: 2.2n, rcl:C-EUC1608
- added R_I2: 1k, user_rcl:R_SHUGOU
Connections:
- removed net N$40: C14.2, C15.2, C16.2, F_C1.2, F_C2.2, F_C6.2, R11.2, R12.2, R13.2, R14.2, R27.1, R28.1, R29.1, R30.1, R31.1, R32.1, U$1.PIN22_CSP, U$1.PIN38_LSS, U$10.PIN3_S, U$12.PIN3_S, U$14.A1, U$14.A2, U$15.A1, U$15.A2, U$18.A1, U$18.A2, U$8.PIN3_S
- new net N$20: C19.1, R_I2.7, R_I2.8, U$1.PIN22_CSP
- new net N$6: C14.2, C15.2, C16.2, F_C1.2, F_C2.2, F_C6.2, R11.2, R12.2, R13.2, R14.2, R27.1, R28.1, R29.1, R30.1, R31.1, R32.1, R_I2.1, R_I2.2, U$1.PIN38_LSS, U$10.PIN3_S, U$12.PIN3_S, U$14.A1, U$14.A2, U$15.A1, U$15.A2, U$18.A1, U$18.A2, U$8.PIN3_S
- new net N$9: C19.2, R_I2.5, R_I2.6, U$1.PIN21_CSN
- net GND: now also R_I2.3, R_I2.4; no longer U$1.PIN21_CSN
Other:
- moved on the sheet: R10, R11, R12, R13, R14, R15, R5, R8, R9
